File: mcxn-proto-card/oresat-proto-card-sch-microcontroller.kicad_sch (KiCad schematic)
At the start: 101 parts, among them U1 MCXN947VKLT, U8 TCAN330, Y2 24 MHz

Commit message: First commit of Science Card
Parts:
- removed TP11, TP17, TP18, TP19, TP20, TP22, TP25, TP26, TP27, TP28, TP29, TP32, TP33, TP41, TP42, TP43, TP44, TP45, TP46, TP47, TP48, TP49, TP5, TP50, TP51, TP54, TP58, TP59, TP60, TP61, TP62, TP63, TP64, TP65, TP66, TP67, TP68, TP69, TP7, TP70, TP71, TP72, TP73, TP74, TP75, TP76, TP77, TP78, TP79, TP8, TP80, TP81, TP82, TP83, TP84, TP85, TP86: Test-Point, oresat-misc:TestPoint-0.75mm-th, symbol oresat-misc:Test-Point-0.75mm-th
- added J10: 61083-061409LF, 61083-061409LF:AMPHENOL_61083-061409LF, symbol Connector_Generic:Conn_01x60
Connections:
- net GND: now also J10.1 (Pin_1), J10.13 (Pin_13), J10.14 (Pin_14), J10.15 (Pin_15), J10.16 (Pin_16), J10.2 (Pin_2), J10.29 (Pin_29), J10.3 (Pin_3), J10.30 (Pin_30), J10.31 (Pin_31), J10.32 (Pin_32), J10.4 (Pin_4), J10.45 (Pin_45), J10.46 (Pin_46), J10.47 (Pin_47), J10.48 (Pin_48), J10.51 (Pin_51), J10.52 (Pin_52), J10.53 (Pin_53), J10.54 (Pin_54), J10.59 (Pin_59), J10.60 (Pin_60)
- net P2_0: now also J10.18 (Pin_18)
- net P2_1: now also J10.22 (Pin_22)
- net P3_10: now also J10.17 (Pin_17)
- net P3_11: now also J10.19 (Pin_19)
- net P3_12: now also J10.25 (Pin_25)
- net P3_13: now also J10.27 (Pin_27)
- net P3_14: now also J10.33 (Pin_33)
- net P3_15: now also J10.35 (Pin_35)
- net P3_16: now also J10.41 (Pin_41)
- net P3_17: now also J10.43 (Pin_43)
- net P3_8: now also J10.9 (Pin_9)
- net P3_9: now also J10.11 (Pin_11)
- net P2_3 renamed CDH_COMM_RX
- net CDH_COMM_RX: now also J10.6 (Pin_6)
- net P2_4 renamed CDH_COMM_TX
- net CDH_COMM_TX: now also J10.20 (Pin_20)
- net P3_0 renamed BOOT_LOAD_IN0
- net BOOT_LOAD_IN0: now also U1.74 (P3_1), J10.42 (Pin_42); no longer U1.75 (P3_0)
- net P3_1 renamed BOOT_LOAD_IN1
- net BOOT_LOAD_IN1: now also U1.75 (P3_0), J10.44 (Pin_44); no longer U1.74 (P3_1)
- net P4_12 renamed FC2_LPUART_RXD
- net P4_13 renamed FC2_LPUART_TXD
- new net VBUSP: J10.55 (Pin_55), J10.56 (Pin_56), J10.57 (Pin_57), J10.58 (Pin_58)
- no-connect marks 4 -> 59
Other:
- note added: "RF Board Connector"
- moved on the sheet: C12, C26, C27, C29, C30, C31, C47, FB1, L3, R15, R23, R8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
