File: mcxn-proto-card/oresat-proto-card.kicad_sch (KiCad schematic)
At the start: 13 parts, among them J1 J-SAMTEC-TFM-120-X1-XXX-D-RA, J2 J-SAMTEC-TFM-110-01-L-D-RA, J3 SM14B-SHLS-TF, J4 2477330-1, J5 2477330-1, J6 2477330-1, J7 U.FL-R-SMT-1(10), J8 U.FL-R-SMT-1(10), J9 U.FL-R-SMT-1(10)

Commit message: First commit of Science Card
Parts:
- removed J2: J-SAMTEC-TFM-110-01-L-D-RA, oresat-connectors:J-SAMTEC-TFM-110-X1-XXX-D-RA, symbol oresat-connectors:J-SAMTEC-TFM-110-01-L-D-RA
- removed J4, J5, J6: 2477330-1, oresat-connectors:J-MOLEX-SMPM-073300-002X, symbol Connector:Conn_Coaxial
- removed J7, J8, J9: U.FL-R-SMT-1(10), Connector_Coaxial:U.FL_Hirose_U.FL-R-SMT-1_Vertical, symbol Connector:Conn_Coaxial
- removed JP1: PINHD-2X5, Connector_PinHeader_2.54mm:PinHeader_2x11_P2.54mm_Vertical, symbol Connector_Generic:Conn_02x11_Odd_Even
- removed JP2: Conn_01x10, Connector_PinHeader_2.54mm:PinHeader_1x10_P2.54mm_Vertical, symbol Connector_Generic:Conn_01x10
- added J14, J15: ESQ-126-12-G-D, ESQ-126-12-G-D:ESQ-126-Y-X-D, symbol ESQ-126-12-G-D:ESQ-126-12-G-D
Connections:
- net +3.3V: now also J14.47, J14.48, J14.49, J14.50, J14.51, J14.52
- net GND: now also J15.29, J15.30, J15.32
- net SPARE31 renamed LPUART_RXD
- net SPARE32 renamed LPUART_TXD
- new net CDH_COMM_RX: J14.1
- new net CDH_COMM_TX: J14.3
- no-connect marks 2 -> 110
Other:
- note removed: "Aux Connector Breakout"
- note removed: "Auxiliary Connector"
- note removed: "Main Connector Breakout"
- note removed: "RF connections and test points"
