File: mcxn-proto-card/oresat-proto-card.kicad_pcb (KiCad board)
At the start: 4 copper layers, 99.8 x 94.6 mm, 201 parts, among them J1 J-SAMTEC-TFM-120-X1-XXX-D-RA, J2 J-SAMTEC-TFM-110-01-L-D-RA, J3 SM14B-SHLS-TF, J4 2477330-1, J5 2477330-1, J6 2477330-1, J7 U.FL-R-SMT-1(10), J8 U.FL-R-SMT-1(10), J9 U.FL-R-SMT-1(10), Q1 DMP2240UDM, Q2 DMP3050LVT-7, Q7 DMP3050LVT-7, Q8 PMV45EN, Q9 PMV45EN, U1 MCXN947VKLT, U10 TPS62111RSA, U11 MIC842LYC5, U12 MIC842LYC5, U2 MAX7310, U3 TS5A21366DCUR, U6 MAX4211FETE, U8 TCAN330, Y2 24 MHz

Commit message: First commit of Science Card
Parts:
- removed J2: J-SAMTEC-TFM-110-01-L-D-RA, oresat-connectors:J-SAMTEC-TFM-110-X1-XXX-D-RA
- removed J4, J5, J6: 2477330-1, oresat-connectors:J-MOLEX-SMPM-073300-002X
- removed J7, J8, J9: U.FL-R-SMT-1(10), Connector_Coaxial:U.FL_Hirose_U.FL-R-SMT-1_Vertical
- removed JP2: Conn_01x10, Connector_PinHeader_2.54mm:PinHeader_1x10_P2.54mm_Vertical
- removed TP11, TP17, TP18, TP19, TP20, TP22, TP25, TP26, TP27, TP28, TP29, TP32, TP33, TP41, TP42, TP43, TP44, TP45, TP46, TP47, TP48, TP49, TP5, TP50, TP51, TP54, TP58, TP59, TP60, TP61, TP62, TP63, TP64, TP65, TP66, TP67, TP68, TP69, TP7, TP70, TP71, TP72, TP73, TP74, TP75, TP76, TP77, TP78, TP79, TP8, TP80, TP81, TP82, TP83, TP84, TP85, TP86: Test-Point, oresat-misc:TestPoint-0.75mm-th
- added J10: 61083-061409LF, 61083-061409LF:AMPHENOL_61083-061409LF, F.Cu at (148.4, 143.2)
- added J11: 436500201, WM1865-ND:CONN_SD-43650-001_02_MOL, F.Cu at (115.5, 138.3)
- added J14: ESQ-126-12-G-D, ESQ-126-12-G-D:ESQ-126-Y-X-D, B.Cu at (182.4, 76.1)
- added J15: ESQ-126-12-G-D, ESQ-126-12-G-D:ESQ-126-Y-X-D, B.Cu at (187.5, 76.1)
- moved TP14 31.8 mm to (105.0, 102.9)
- moved TP12 31.6 mm to (105.0, 100.1)
- moved D3 26.2 mm to (109.0, 144.7)
- moved D6 26.2 mm to (110.7, 144.7)
- moved D7 26.2 mm to (107.3, 144.7)
- moved R17 26.2 mm to (110.7, 142.0)
- moved R3 26.2 mm to (109.0, 142.0)
- moved R76 26.2 mm to (107.3, 142.0)
- moved D4 26.1 mm to (112.3, 144.7)
- moved R21 26.1 mm to (112.3, 142.0)
- moved TP10 21.4 mm to (105.0, 97.4)
- moved TP9 21.0 mm to (105.0, 94.5)
- moved TP30 13.5 mm to (110.8, 74.2)
- moved TP57 10.4 mm to (113.0, 102.9)
- moved TP55 7.22 mm to (108.0, 102.9)
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Connections:
- net /Microcontroller/P2_3 renamed /Microcontroller/CDH_COMM_RX
- net /Microcontroller/P2_4 renamed /Microcontroller/CDH_COMM_TX
- net /Microcontroller/P3_0 renamed /Microcontroller/BOOT_LOAD_IN1
- net /Microcontroller/P3_1 renamed /Microcontroller/BOOT_LOAD_IN0
- J1 pad 31: /SPARE31 -> /Microcontroller/FC2_0
- J1 pad 32: /SPARE32 -> /Microcontroller/FC2_1
- JP1 pad 17: /SPARE32 -> /Microcontroller/FC2_1
- JP1 pad 22: /SPARE31 -> /Microcontroller/FC2_0
- U1 pad 35: /Microcontroller/P4_12 -> /Microcontroller/FC2_0
- U1 pad 36: /Microcontroller/P4_13 -> /Microcontroller/FC2_1
Routing:
- net /Microcontroller/CDH_COMM_RX: track 20.1 -> 204.7 mm, vias 1 -> 3
- net /Microcontroller/CDH_COMM_TX: track 16.6 -> 199.7 mm, vias 1 -> 5
- net +3.3V: track 44.9 -> 150.4 mm, vias 42 -> 45
- net /Microcontroller/P2_1: track 11.4 -> 101.8 mm, vias 1 -> 3
- net /Microcontroller/P2_0: track 13.1 -> 103.5 mm, vias 1 -> 3
- net /Microcontroller/P3_9: track 13.8 -> 91.2 mm, vias 0 -> 5
- net /Microcontroller/P3_10: track 10.2 -> 86.8 mm, vias 0 -> 4
- net /Microcontroller/P3_11: track 15.0 -> 88.9 mm, vias 0 -> 4
- net /Microcontroller/P3_15: track 17.3 -> 90.5 mm, vias 1 -> 4
- net /Microcontroller/P3_8: track 17.2 -> 90.1 mm, vias 0 -> 4
- net /Microcontroller/P3_16: track 14.0 -> 85.0 mm, vias 1 -> 4
- net /Microcontroller/P3_13: track 16.5 -> 85.2 mm, vias 1 -> 4
- net /Microcontroller/P3_17: track 15.4 -> 84.0 mm, vias 1 -> 4
- net /Microcontroller/FC2_0: track 0.00 -> 67.0 mm, vias 0 -> 5
- net /Microcontroller/P3_12: track 20.1 -> 86.0 mm, vias 1 -> 4
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Other:
- board text removed: "+3.3V"
- board text removed: "OreSat Proto-Card v${REVISION}"

Commit message: Added power P3.3V planes
Connections:
- U10 pad 17: GND -> +3.3V
- U11 pad 2: GND -> +3.3V
- U2 pad 17: GND -> +3.3V
- U6 pad 17: GND -> +3.3V
Routing:
- net +3.3V: track 150.4 -> 44.7 mm, vias 45 -> 53
- net VBUSP: track 53.3 -> 15.8 mm, vias 9 -> 11
- net GND: track 1.42 -> 0.00 mm, vias 318 -> 311
- net /Microcontroller/P3_9: track 91.2 -> 90.7 mm, vias 5 -> 4
- net unconnected-(J10-Pin_10-Pad10): vias 1 -> 0
