File: mcxn-proto-card/oresat-proto-card-sch-power.kicad_sch (KiCad schematic)
At the start: 87 parts, among them Q1 DMP2240UDM, Q2 DMP3050LVT-7, Q7 DMP3050LVT-7, Q8 PMV45EN, Q9 PMV45EN, U10 TPS62111RSA, U11 MIC842LYC5, U12 MIC842LYC5, U2 MAX7310, U3 TS5A21366DCUR, U6 MAX4211FETE

Commit message: First commit of Science Card
Parts:
- added J11: 436500201, WM1865-ND:CONN_SD-43650-001_02_MOL, symbol 436500201:436500201
Connections:
- net GND: now also J11.2
- net VBUSP: now also J11.1
Other:
- note added: "SDR Power Connector"

Commit message: Finalized design with adding properly measured mounting holes that line up with piPlasma. As well as changing sense resistor to allow 1A trip
Parts:
- R64: value 100m -> 30m; DPN CSR1206FKR100CT-ND -> CSR1206FK30L0TR-ND; MPN CSR1206FKR100 -> CSR1206FK30L0
Other:
- note added: "Feedback settings trips at 985mA"
- note removed: "Feedback settings trips at 295m mA"
Changed lines of the file:
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@@
 		)
 	)
-	(text "Feedback settings trips at 295m mA"
+	(text "Feedback settings trips at 985mA"
 		(exclude_from_sim no)
 		(at 299.212 53.848 0)
@@
 			)
 		)
-		(property "Value" "100m"
+		(property "Value" "30m"
 			(at 268.478 42.926 90)
 			(show_name no)
@@
 			)
 		)
-		(property "Description" "100 mOhms ±1% 0.5W, 1/2W Chip Resistor 1206 (3216 Metric) Current Sense Thick Film"
+		(property "Description" "RES 0.03 OHM 1% 1/2W 1206"
 			(at 267.97 44.45 0)
 			(hide yes)
@@
 			)
 		)
-		(property "DPN" "CSR1206FKR100CT-ND"
+		(property "DPN" "CSR1206FK30L0TR-ND"
 			(at 267.97 44.45 0)
 			(hide yes)
@@
 			)
 		)
-		(property "MPN" "CSR1206FKR100"
+		(property "MPN" "CSR1206FK30L0"
 			(at 267.97 44.45 0)
 			(hide yes)
